Commit message: updating models:

File: models/iiwa14_primitive_collision.urdf (robot description, URDF)
Before this commit: robot iiwa14, 11 links, 10 joints
Links:
- link iiwa_link_7: geometry collision cylinder length=0.1 radius=0.05585650291; visual mesh filename=package://drake_models/iiwa_description/meshes/iiwa14/visua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
