Commit message: checkpointing

File: clutter_example/models/planar_iiwa14_spheres_dense_elbow_collision.urdf (robot description, URDF)
Before this commit: robot iiwa14, 11 links, 10 joints
Links:
- removed link base
- link iiwa_link_1: geometry collision sphere radius=0.07959901601; visual mesh filename=package://drake_models/iiwa_description/meshes/iiwa14/visua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
- link iiwa_link_2: geometry collision sphere radius=0.06602481863; collision sphere radius=0.07959901601
- link iiwa_link_3: geometry collision sphere radius=0.055; collision sphere radius=0.055
- link iiwa_link_4: geometry collision sphere radius=0.06; collision sphere radius=0.06
- link iiwa_link_5: geometry visual mesh filename=package://drake_models/iiwa_description/meshes/iiwa14/visua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; visual mesh filename=package://drake_models/iiwa_description/meshes/iiwa14/visua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
- link iiwa_link_6: geometry collision sphere radius=0.055; collision sphere radius=0.08
- link iiwa_link_7: geometry collision sphere radius=0.06; visual mesh filename=package://drake_models/iiwa_description/meshes/iiwa14/visua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
Joints:
- removed joint iiwa_base_joint
- joint iiwa_joint_1: axis 0 0 1 -> (none); limit lower=-2.96705972839 upper=2.96705972839 effort=320 velocity=1.4835298641951802 -> (none); type revolute -> fixed
- joint iiwa_joint_3: axis 0 0 1 -> (none); limit lower=-2.96705972839 upper=2.96705972839 effort=176 velocity=1.7453292519943295 -> (none); type revolute -> fixed
- joint iiwa_joint_5: axis 0 0 1 -> (none); limit lower=-2.96705972839 upper=2.96705972839 effort=110 velocity=2.2689280275926285 -> (none); type revolute -> fixed
- joint iiwa_joint_7: axis 0 0 1 -> (none); limit lower=-3.05432619099 upper=3.05432619099 effort=40 velocity=2.356194490192345 -> (none); origin xyz=0 0.081 0 rpy=-1.570796326794897 3.141592653589793 0 -> xyz=0 0.081 0 rpy=-1.570796326794897 -1.57079632679 0; type revolute -> fixed

File: models/iiwa14_spheres_cylinders_collision.urdf (robot description, URDF)
Before this commit: robot iiwa14, 11 links, 10 joints
Links:
- link iiwa_link_5: geometry collision sphere radius=0.05281876964; collision sphere radius=0.06644602201
- link iiwa_link_6: geometry collision sphere radius=0.06341754633; visual mesh filename=package://drake_models/iiwa_description/meshes/iiwa14/visua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
